File: Tavern64.kicad_pcb (KiCad board)
At the start: 2 copper layers, 314.3 x 100 mm, 159 parts, among them SW1 MX_SW_HS_LED, SW10 MX_SW_HS_LED, SW102 SW_PUSH, SW11 MX_SW_HS_LED, SW12 MX_SW_HS_LED, SW13 MX_SW_HS_LED, SW14 MX_SW_HS_LED, SW15 MX_SW_HS_LED, SW16 MX_SW_HS_LED, SW17 MX_SW_HS_LED, SW18 MX_SW_HS_LED, SW19 MX_SW_HS_LED, SW2 MX_SW_HS_LED, SW20 MX_SW_HS_LED, SW21 MX_SW_HS_LED, SW22 MX_SW_HS_LED, SW23 MX_SW_HS_LED, SW24 MX_SW_HS_LED, SW25 MX_SW_HS_LED, SW26 MX_SW_HS_LED, SW27 MX_SW_HS_LED, SW28 MX_SW_HS_LED, SW29 MX_SW_HS, SW3 MX_SW_HS_LED, SW30 MX_SW_HS_LED, SW31 MX_SW_HS_LED, SW32 MX_SW_HS_LED, SW33 MX_SW_HS_LED, SW34 MX_SW_HS_LED, SW35 MX_SW_HS_LED, SW36 MX_SW_HS_LED, SW37 MX_SW_HS_LED, SW38 MX_SW_HS_LED, SW39 MX_SW_HS_LED, SW4 MX_SW_HS_LED, SW40 MX_SW_HS_LED, SW41 MX_SW_HS_LED, SW42 MX_SW_HS_LED, SW43 MX_SW_HS, SW44 MX_SW_HS_LED, SW45 MX_SW_HS_LED, SW46 MX_SW_HS_LED, SW47 MX_SW_HS_LED, SW48 MX_SW_HS_LED, SW49 MX_SW_HS_LED, SW5 MX_SW_HS_LED, SW50 MX_SW_HS_LED, SW51 MX_SW_HS_LED, SW52 MX_SW_HS_LED, SW53 MX_SW_HS_LED, SW54 MX_SW_HS_LED, SW55 MX_SW_HS_LED, SW56 MX_SW_HS_LED, SW57 MX_SW_HS, SW58 MX_SW_HS_LED, SW59 MX_SW_HS_LED, SW6 MX_SW_HS_LED, SW60 MX_SW_HS_LED, SW61 MX_SW_HS_LED, SW62 MX_SW_HS_LED, SW63 MX_SW_HS_LED, SW64 MX_SW_HS_LED, SW65 MX_SW_HS_LED, SW66 MX_SW_HS_LED, SW67 MX_SW_HS_LED, SW7 MX_SW_HS_LED, SW8 MX_SW_HS_LED, SW9 MX_SW_HS_LED, U1 Rasbperry Pi Pico RP2040 Purp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

Commit message: Add files via upload
Parts:
- added H1: MountingHole, Oden Library:MountingHole_2.2mm_M2_Pad, B.Cu at (111.1, 79.8)
- added H2: MountingHole, Oden Library:MountingHole_2.2mm_M2_Pad, B.Cu at (159.5, 136.9)
- added H3: MountingHole, Oden Library:MountingHole_2.2mm_M2_Pad, B.Cu at (275.4, 130.2)
- added H4: MountingHole, Oden Library:MountingHole_2.2mm_M2_Pad, B.Cu at (345.3, 75.4)
- added H5: MountingHole, Oden Library:MountingHole_2.2mm_M2_Pad, B.Cu at (61.0, 146.6)
- added H6: MountingHole, Oden Library:MountingHole_2.2mm_M2_Pad, B.Cu at (371.0, 146.6)
- added H7: MountingHole, Oden Library:MountingHole_2.2mm_M2_Pad, B.Cu at (371.0, 51.0)
- added L4: ~, Oden Library:SK6812MINI-E, F.Cu at (273.8, 137.7)
- added REF**: STAB_MX_2u, marbastlib-mx:STAB_MX_2u, F.Cu at (254.0, 136.9)
- added REF**: STAB_MX_2u, marbastlib-mx:STAB_MX_2u, F.Cu at (215.9, 136.9)
- SW58, SW59: footprint Oden Library:CherryMX_Choc_Hotswap v2 with LEDs -> Oden Library:CherryMX_Choc_Hotswap v2 with LEDs shortened
- SW63: footprint Oden Library:CherryMX_Choc_Hotswap v2 with LEDs -> Oden Library:CherryMX_Choc_Hotswap v2 for spacebar
- moved R2 0.41 mm to (363.4, 115.1)
- renumbered U3 to L2, U2 to L3
Connections:
- ENC1 pad B: ENC 1B -> ENC B
- ENC2 pad B: ENC 2B -> ENC B
- ENC3 pad B: ENC 3B -> ENC B
- IND1 pad 2: IND LED -> IND SCRL
- IND2 pad 2: IND LED -> IND CAPS
- IND3 pad 2: IND LED -> IND NUML
- L3 pad 2L: Net-(SW63-DIN) -> Net-(L3-DOUT)
- SW64 pad 4L: Net-(SW63-DOUT) -> Net-(L4-DOUT)
- U1 pad 17: ENC 1B -> ENC 1A
- U1 pad 18: ENC 1A -> ENC 3A
- U1 pad 19: ENC 2B -> ENC 2A
- U1 pad 20: ENC 2A -> ENC B
- U1 pad 21: ENC 3B -> ROW 4
- U1 pad 22: ENC 3A -> ROW 3
- U1 pad 23: ROW 4 -> ROW 2
- U1 pad 24: ROW 3 -> ROW 1
- U1 pad 25: ROW 2 -> ROW 0
- U1 pad 26: ROW 1 -> IND NUML
- U1 pad 27: ROW 0 -> IND CAPS
- U1 pad 28: IND LED -> IND SCRL
Routing:
- net ENC B: track 0.00 -> 72.2 mm
- net Net-(SW63-DOUT): track 68.9 -> 0.00 mm, vias 4 -> 0
- net Net-(L3-DOUT): track 0.00 -> 55.6 mm
- net Net-(SW63-DIN): track 43.3 -> 0.00 mm, vias 2 -> 0
- net Net-(L4-DOUT): track 0.00 -> 40.2 mm, vias 0 -> 2
- net ENC 3B: track 36.2 -> 0.00 mm
- net ENC 2B: track 28.1 -> 0.00 mm
- net GND: track 2059.7 -> 2085.5 mm, vias 131 -> 228
- net COL 2: track 179.8 -> 202.1 mm
- net ENC 3A: track 47.0 -> 67.6 mm
- net IND LED: track 18.6 -> 0.00 mm
- net IND NUML: track 0.00 -> 17.7 mm
- net ENC 2A: track 28.1 -> 45.6 mm
- net IND CAPS: track 0.00 -> 11.1 mm
- net ROW 3: track 354.6 -> 345.2 mm
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- added copper zone on B.Cu, net GND
- added copper zone on F.Cu, net GND
Other:
- board text added: "Designed by Jacob Thompson 2023"
- board text added: "JLCJLCJLCJLC"
- board text added: "Tavern64"
