File: Tavern64.kicad_sch (KiCad schematic)
At the start: 153 parts, among them SW1 MX_SW_HS_LED, SW10 MX_SW_HS_LED, SW102 SW_PUSH, SW11 MX_SW_HS_LED, SW12 MX_SW_HS_LED, SW13 MX_SW_HS_LED, SW14 MX_SW_HS_LED, SW15 MX_SW_HS_LED, SW16 MX_SW_HS_LED, SW17 MX_SW_HS_LED, SW18 MX_SW_HS_LED, SW19 MX_SW_HS_LED, SW2 MX_SW_HS_LED, SW20 MX_SW_HS_LED, SW21 MX_SW_HS_LED, SW22 MX_SW_HS_LED, SW23 MX_SW_HS_LED, SW24 MX_SW_HS_LED, SW25 MX_SW_HS_LED, SW26 MX_SW_HS_LED, SW27 MX_SW_HS_LED, SW28 MX_SW_HS_LED, SW29 MX_SW_HS, SW3 MX_SW_HS_LED, SW30 MX_SW_HS_LED, SW31 MX_SW_HS_LED, SW32 MX_SW_HS_LED, SW33 MX_SW_HS_LED, SW34 MX_SW_HS_LED, SW35 MX_SW_HS_LED, SW36 MX_SW_HS_LED, SW37 MX_SW_HS_LED, SW38 MX_SW_HS_LED, SW39 MX_SW_HS_LED, SW4 MX_SW_HS_LED, SW40 MX_SW_HS_LED, SW41 MX_SW_HS_LED, SW42 MX_SW_HS_LED, SW43 MX_SW_HS, SW44 MX_SW_HS_LED, SW45 MX_SW_HS_LED, SW46 MX_SW_HS_LED, SW47 MX_SW_HS_LED, SW48 MX_SW_HS_LED, SW49 MX_SW_HS_LED, SW5 MX_SW_HS_LED, SW50 MX_SW_HS_LED, SW51 MX_SW_HS_LED, SW52 MX_SW_HS_LED, SW53 MX_SW_HS_LED, SW54 MX_SW_HS_LED, SW55 MX_SW_HS_LED, SW56 MX_SW_HS_LED, SW57 MX_SW_HS, SW58 MX_SW_HS_LED, SW59 MX_SW_HS_LED, SW6 MX_SW_HS_LED, SW60 MX_SW_HS_LED, SW61 MX_SW_HS_LED, SW62 MX_SW_HS_LED, SW63 MX_SW_HS_LED, SW64 MX_SW_HS_LED, SW65 MX_SW_HS_LED, SW66 MX_SW_HS_LED, SW67 MX_SW_HS_LED, SW7 MX_SW_HS_LED, SW8 MX_SW_HS_LED, SW9 MX_SW_HS_LED, U1 Rasbperry Pi Pico RP2040 Purp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

Commit message: Add files via upload
Parts:
- added H1, H2, H3, H4, H5, H6, H7: MountingHole, Oden Library:MountingHole_2.2mm_M2_Pad, symbol Mechanical:MountingHole
- added L4: ~, Oden Library:SK6812MINI-E, symbol Oden library:SK6812MINI-E
- renumbered U3 to L2, U2 to L3
Connections:
- net ENC 1A: now also U1.17 (GP14); no longer U1.18 (GP15)
- net ENC 2A: now also U1.19 (GP16); no longer U1.20 (GP17)
- net ENC 3A: now also U1.18 (GP15); no longer U1.22 (GP19)
- net GND: now also L4.3L (GND); no longer SW63.3L (GND)
- net POWER: now also L4.1L (VDD); no longer SW63.1L (VDD)
- net ROW 0: now also U1.25 (GP22); no longer U1.27 (GP24)
- net ROW 1: now also U1.24 (GP21); no longer U1.26 (GP23)
- net ROW 2: now also U1.23 (GP20); no longer U1.25 (GP22)
- net ROW 3: now also U1.22 (GP19); no longer U1.24 (GP21)
- net ROW 4: now also U1.21 (GP18); no longer U1.23 (GP20)
- net at SW64.4L (DIN): now also L4.2L (DOUT); no longer SW63.2L (DOUT)
- net at L3.2L (DOUT): now also L4.4L (DIN); no longer SW63.4L (DIN)
- net ENC 1B renamed ENC B
- net ENC B: now also ENC2.B, ENC3.B, U1.20 (GP17); no longer U1.17 (GP14)
- removed net ENC 2B: ENC2.B, U1.19 (GP16)
- removed net ENC 3B: ENC3.B, U1.21 (GP18)
- net IND LED renamed IND SCRL
- net IND SCRL: no longer IND2.2 (A), IND3.2 (A)
- new net IND CAPS: IND2.2 (A), U1.27 (GP24)
- new net IND NUML: IND3.2 (A), U1.26 (GP23)
